File: pcbs/4_Key/Seismos_4-Key/Seismos_4-Key.kicad_pcb (KiCad board)
At the start: 2 copper layers, 19 x 86.4 mm, 10 parts, among them J1 SM09B-SRSS-TB(LF)(SN), SW1 Switch_SK6812-E_Diode, SW2 Switch_SK6812-E_Diode, SW3 Switch_SK6812-E_Diode, SW4 Switch_SK6812-E_Diode

Commit message: Fix 4Key Column Hole Size
Converted the M3 holes to the standard footprint instead of edge cut
layer drawing of a circle. Also updated names of gerber output folders.
Parts:
- added REF**: Hole_M3_3.2mm, Seismos-libs:Hole_M3_3.2mm, F.Cu at (53.5, 108.5)
- added REF**: Hole_M3_3.2mm, Seismos-libs:Hole_M3_3.2mm, F.Cu at (40.5, 108.5)
Other:
- outline, holes or cut-outs redrawn
Changed lines of the file:
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@@
       (drillshape 0)
       (scaleselection 1)
-      (outputdirectory "Export/")
+      (outputdirectory "Seismos_4Key_gbr/")
     )
   )
@@
     )
   )
+  (footprint "Seismos-libs:Hole_M3_3.2mm" (layer "F.Cu")
+    (at 53.5 108.5)
+    (attr smd)
+    (fp_text reference "REF**" (at 0 -0.5 unlocked) (layer "Cmts.User")
+        (effects (font (size 1 1) (thickness 0.1)))
+    )
+    (fp_text value "Hole_M3_3.2mm" (at 0 1 unlocked) (layer "F.Fab")
+        (effects (font (size 1 1) (thickness 0.15)))
+    )
+    (fp_text user "${REFERENCE}" (at 0 2.5 unlocked) (layer "F.Fab")
+        (effects (font (size 1 1) (thickness 0.15)))
+    )
+    (pad "" np_thru_hole circle (at 0 0) (size 3.2 3.2) (drill 3.2) (layers "F&B.Cu" "*.Mask"))
+  )
+  (footprint "Seismos-libs:Hole_M3_3.2mm" (layer "F.Cu")
+    (at 40.5 108.5)
+    (attr smd)
+    (fp_text reference "REF**" (at 0 -0.5 unlocked) (layer "Cmts.User")
+        (effects (font (size 1 1) (thickness 0.1)))
+    )
+    (fp_text value "Hole_M3_3.2mm" (at 0 1 unlocked) (layer "F.Fab")
+        (effects (font (size 1 1) (thickness 0.15)))
+    )
+    (fp_text user "${REFERENCE}" (at 0 2.5 unlocked) (layer "F.Fab")
+        (effects (font (size 1 1) (thickness 0.15)))
+    )
+    (pad "" np_thru_hole circle (at 0 0) (size 3.2 3.2) (drill 3.2) (layers "F&B.Cu" "*.Mask"))
+  )
   (footprint "Diode_SMD:D_SOD-123" (layer "B.Cu")
     (at 39.5 56 -90)
@@
   (gr_line (start 37.5 31) (end 40.3 31)
     (stroke (width 0.1) (type default)) (layer "Edge.Cuts"))
-  (gr_circle (center 53.5 108.5) (end 55 108.5)
-    (stroke (width 0.1) (type default)) (fill none) (layer "Edge.Cuts"))
   (gr_line (start 56.5 31) (end 53.7 31)
     (stroke (width 0.1) (type default)) (layer "Edge.Cuts"))
@@
   (gr_line (start 53.7 31) (end 53.7 25)
     (stroke (width 0.1) (type default)) (layer "Edge.Cuts"))
-  (gr_circle (center 40.5 108.5) (end 42 108.5)
-    (stroke (width 0.1) (type default)) (fill none) (layer "Edge.Cuts"))
   (gr_line (start 40.3 25) (end 53.7 25)
     (stroke (width 0.1) (type default)) (layer "Edge.Cuts"))
