File: pcbs/4_Key/Seismos_4-Thumb/Seismos_4-Thumb.kicad_pcb (KiCad board)
At the start: 2 copper layers, 38 x 48.4 mm, 9 parts, among them J1 SM09B-SRSS-TB(LF)(SN), SW1 Switch_SK6812-E_Diode, SW2 Switch_SK6812-E_Diode, SW3 Switch_SK6812-E_Diode, SW4 Switch_SK6812-E_Diode

Commit message: Completed Thumb 2x2 module
Parts:
- added REF**: Hole_M3_3.2mm, Seismos-libs:Hole_M3_3.2mm, F.Cu at (40.5, 70.5)
- added REF**: Hole_M3_3.2mm, Seismos-libs:Hole_M3_3.2mm, F.Cu at (72.5, 70.5)
Routing:
- net /Col_In: track 0.00 -> 101.2 mm, vias 0 -> 3
- net /V+: track 0.00 -> 70.5 mm, vias 0 -> 4
- net Net-(SW3B-DOUT): track 0.00 -> 36.4 mm
- net /Row2: track 0.00 -> 34.9 mm, vias 0 -> 1
- net /Row3: track 0.00 -> 29.1 mm, vias 0 -> 1
- net GND: track 0.00 -> 21.8 mm, vias 0 -> 4
- net Net-(SW1B-DOUT): track 0.00 -> 19.6 mm
- net /Row1: track 0.00 -> 16.8 mm, vias 0 -> 1
- net /RGB_In: track 0.00 -> 16.4 mm, vias 0 -> 1
- net Net-(SW2B-DOUT): track 0.00 -> 15.8 mm
- net /RGB_Out: track 0.00 -> 14.3 mm, vias 0 -> 1
- net Net-(D4-A): track 0.00 -> 6.50 mm
- net Net-(D3-A): track 0.00 -> 6.50 mm
- net Net-(D2-A): track 0.00 -> 6.50 mm
- net Net-(D1-A): track 0.00 -> 6.50 mm
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- added copper zone on B.Cu, net GND
- added copper zone on F.Cu, net GND
Other:
- outline, holes or cut-outs redrawn
