File: pcbs/Switch PCBs (Plates)/4_Key/Seismos_4-Thumb/Seismos_4-Thumb.kicad_sch (KiCad schematic)
At the start: 9 parts, among them J1 SM10B-SRSS-TB(LF)(SN), SW1 Switch_SK6812-E_Diode, SW2 Switch_SK6812-E_Diode, SW3 Switch_SK6812-E_Diode, SW4 Switch_SK6812-E_Diode

Commit message: Fix schematic reference errors for thumb
Errors appeared when applying thumb schematic to PCB.
This doesn't change the PCB footprints though, so no re-release
Parts:
- SW1, SW2, SW3, SW4: footprint KeysOnRails-lib:Switch_SK6812-E_Diode -> Seismos-libs:Switch_SK6812-E_Diode
- SW1, SW2, SW3, SW4: footprint Seismos-lib:Switch_SK6812-E_Diode -> Seismos-libs:Switch_SK6812-E_Diode
Changed lines of the file:
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@@
     )
   )
-  (symbol (lib_name "Switch_SK6812-E_Diode_1") (lib_id "Seismos-sym:Switch_SK6812-E_Diode") (at 210.82 45.72 0) (unit 2)
+  (symbol (lib_id "Seismos-sym:Switch_SK6812-E_Diode") (at 210.82 45.72 0) (unit 2)
     (in_bom yes) (on_board yes) (dnp no) (fields_autoplaced)
     (property "Reference" "SW1" (at 210.82 34.29 0)
@@
       (effects (font (size 1.27 1.27)))
     )
-    (property "Footprint" "KeysOnRails-lib:Switch_SK6812-E_Diode" (at 210.82 36.83 0)
+    (property "Footprint" "Seismos-libs:Switch_SK6812-E_Diode" (at 210.82 36.83 0)
       (effects (font (size 1.27 1.27)) hide)
     )
@@
       (effects (font (size 1.27 1.27)))
     )
-    (property "Footprint" "Seismos-lib:Switch_SK6812-E_Diode" (at 104.14 52.07 0)
+    (property "Footprint" "Seismos-libs:Switch_SK6812-E_Diode" (at 104.14 52.07 0)
       (effects (font (size 1.27 1.27)) hide)
     )
@@
     )
   )
-  (symbol (lib_name "Switch_SK6812-E_Diode_2") (lib_id "Seismos-sym:Switch_SK6812-E_Diode") (at 210.82 106.68 0) (unit 2)
+  (symbol (lib_id "Seismos-sym:Switch_SK6812-E_Diode") (at 210.82 106.68 0) (unit 2)
     (in_bom yes) (on_board yes) (dnp no) (fields_autoplaced)
     (property "Reference" "SW4" (at 210.82 95.25 0)
@@
       (effects (font (size 1.27 1.27)))
     )
-    (property "Footprint" "KeysOnRails-lib:Switch_SK6812-E_Diode" (at 210.82 97.79 0)
+    (property "Footprint" "Seismos-libs:Switch_SK6812-E_Diode" (at 210.82 97.79 0)
       (effects (font (size 1.27 1.27)) hide)
     )
@@
     )
   )
-  (symbol (lib_name "Switch_SK6812-E_Diode_3") (lib_id "Seismos-sym:Switch_SK6812-E_Diode") (at 210.82 66.04 0) (unit 2)
+  (symbol (lib_id "Seismos-sym:Switch_SK6812-E_Diode") (at 210.82 66.04 0) (unit 2)
     (in_bom yes) (on_board yes) (dnp no) (fields_autoplaced)
     (property "Reference" "SW2" (at 210.82 54.61 0)
@@
       (effects (font (size 1.27 1.27)))
     )
-    (property "Footprint" "KeysOnRails-lib:Switch_SK6812-E_Diode" (at 210.82 57.15 0)
+    (property "Footprint" "Seismos-libs:Switch_SK6812-E_Diode" (at 210.82 57.15 0)
       (effects (font (size 1.27 1.27)) hide)
     )
@@
     )
   )
-  (symbol (lib_name "Switch_SK6812-E_Diode_4") (lib_id "Seismos-sym:Switch_SK6812-E_Diode") (at 210.82 86.36 0) (unit 2)
+  (symbol (lib_id "Seismos-sym:Switch_SK6812-E_Diode") (at 210.82 86.36 0) (unit 2)
     (in_bom yes) (on_board yes) (dnp no) (fields_autoplaced)
     (property "Reference" "SW3" (at 210.82 74.93 0)
@@
       (effects (font (size 1.27 1.27)))
     )
-    (property "Footprint" "KeysOnRails-lib:Switch_SK6812-E_Diode" (at 210.82 77.47 0)
+    (property "Footprint" "Seismos-libs:Switch_SK6812-E_Diode" (at 210.82 77.47 0)
       (effects (font (size 1.27 1.27)) hide)
     )
@@
       (effects (font (size 1.27 1.27)))
     )
-    (property "Footprint" "Seismos-lib:Switch_SK6812-E_Diode" (at 104.14 31.75 0)
+    (property "Footprint" "Seismos-libs:Switch_SK6812-E_Diode" (at 104.14 31.75 0)
       (effects (font (size 1.27 1.27)) hide)
     )
@@
       (effects (font (size 1.27 1.27)))
     )
-    (property "Footprint" "Seismos-lib:Switch_SK6812-E_Diode" (at 104.14 72.39 0)
+    (property "Footprint" "Seismos-libs:Switch_SK6812-E_Diode" (at 104.14 72.39 0)
       (effects (font (size 1.27 1.27)) hide)
     )
@@
       (effects (font (size 1.27 1.27)))
     )
-    (property "Footprint" "Seismos-lib:Switch_SK6812-E_Diode" (at 104.14 92.71 0)
-      (effects (font (size 1.27 1.27)) hide)
-    )
+    (property "Footprint" "Seismos-libs:Switch_SK6812-E_Diode" (at 104.14 92.71 0)
+      (effects (font (size 1.27 1.27)) hide)
+    )
