File: pcbs/Core PCBs (Mantles)/5 Key Core/Seismos_5CoreR/Seismos_5CoreR.kicad_pcb (KiCad board)
At the start: 2 copper layers, 147 x 78 mm, 30 parts, among them J1 SM09B-SRSS-TB(LF)(SN), J2 SM09B-SRSS-TB(LF)(SN), J3 SM09B-SRSS-TB(LF)(SN), J4 SM09B-SRSS-TB(LF)(SN), J5 SM09B-SRSS-TB(LF)(SN), J6 SM09B-SRSS-TB(LF)(SN), J7 SM09B-SRSS-TB(LF)(SN), J8 MJ-4PP-9-Lily58, J9 Conn_01x05_Pin, SW1 RotaryEncoder_Switch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

Commit message: Fix right encoder button, fix connector refs
Right side encoder was still connected to the 6th column for some
reason... Figures when you copy paste the same board design into a
different project.

Also fixed references for the SH connectors, so it doesn't look weird
Parts:
- J1, J2, J3, J4, J5, J6: value SM09B-SRSS-TB(LF)(SN) -> SM010B-SRSS-TB(LF)(SN)
Connections:
- SW1 pad S2: /Col_In6 -> /Col_InT
Routing:
- net /Col_In6: track 177.7 -> 145.3 mm, vias 3 -> 2
- net /Col_InT: track 49.2 -> 60.9 mm, vias 0 -> 1
Other:
- board text added: "Rev. 1.1.2"
- board text removed: "Rev. 1.1.1"
