File: pcbs/Core PCBs (Mantles)/5 Key Core/Seismos_5CoreR/Seismos_5CoreR.kicad_pcb (KiCad board)
At the start: 2 copper layers, 147 x 78 mm, 30 parts, among them J1 SM010B-SRSS-TB(LF)(SN), J2 SM010B-SRSS-TB(LF)(SN), J3 SM010B-SRSS-TB(LF)(SN), J4 SM010B-SRSS-TB(LF)(SN), J5 SM010B-SRSS-TB(LF)(SN), J6 SM010B-SRSS-TB(LF)(SN), J7 SM09B-SRSS-TB(LF)(SN), J8 MJ-4PP-9-Lily58, J9 Conn_01x05_Pin, SW1 RotaryEncoder_Switch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

Commit message: Added 74HC595A support, new release
New PCB versions supporting shift register.
Another JST SH connector is added to expose 2 spare pins.

Footprints for microcontroller were updated using modified footprint from library.
Original variants updated to these new footprints with some fixes as well.
Parts:
- J7: value SM09B-SRSS-TB(LF)(SN) -> SM10B-SRSS-TB_(LF)(SN)
- U1: footprint keyboard_reversible:ProMicro -> Seismos-libs:keebRev-onesided_ProMicro
Routing:
- net /RGB_In7: track 177.6 -> 175.5 mm
Other:
- board text added: "Rev. 2.0.0"
- board text removed: "Rev. 1.1.2"

Commit message: HOTFIX, power switch bridges to ground
Connections:
- U2 pad L1: GND -> unconnected-(U2-PadL1)
Routing:
- net GND: track 396.7 -> 395.0 mm

Commit message: Update PCB version and gerbers for HOTFIX
Other:
- board text added: "Rev. 2.1.0"
- board text removed: "Rev. 2.0.0"
Changed lines of the file:
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@@
 		(layer "Edge.Cuts")
 	)
-	(gr_text "Rev. 2.0.0"
+	(gr_text "Rev. 2.1.0"
 		(at 53.45 78.9 90)
 		(layer "B.SilkS")
