File: pcbs/Core PCBs (Mantles)/5 Key Core/Seismos_5CoreR/Seismos_5CoreR.kicad_sch (KiCad schematic)
At the start: 21 parts, among them J1 SM09B-SRSS-TB(LF)(SN), J2 SM09B-SRSS-TB(LF)(SN), J3 SM09B-SRSS-TB(LF)(SN), J4 SM09B-SRSS-TB(LF)(SN), J5 SM09B-SRSS-TB(LF)(SN), J6 SM09B-SRSS-TB(LF)(SN), J7 SM09B-SRSS-TB(LF)(SN), J8 MJ-4PP-9-Lily58, J9 Conn_01x05_Pin, SW1 RotaryEncoder_Switch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

Commit message: Release v1.1.1
Added I2C pull up resistors and bridge contacts on the backif 5V power
is desired. If you have v1.1, V+ is actually close to the headphone
jack, so you can scratch off the trace and bridge there.
Parts:
- added JP1: Jumper_2_Open, Jumper:SolderJumper-2_P1.3mm_Open_TrianglePad1.0x1.5mm, symbol Seismos-sym:Jumper_2_Open
- added R1, R2: R, Resistor_SMD:R_0603_1608Metric_Pad0.98x0.95mm_HandSolder, symbol Seismos-sym:Resistor
Connections:
- net SCL: now also R2.2
- net SDA: now also R1.2
- net V+: now also JP1.2 (B), R1.1, R2.1
- net at J8.1: now also JP1.1 (A)
Changed lines of the file:
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@@
+    (stroke (width 0) (type default))
+  )
+  (wire (pts (xy 297.18 160.02) (xy 297.18 165.1))
     (stroke (width 0) (type default))
   )
@@
     (stroke (width 0) (type default))
   )
+  (wire (pts (xy 304.8 160.02) (xy 304.8 165.1))
+    (stroke (width 0) (type default))
+  )
   (wire (pts (xy 115.57 80.01) (xy 115.57 82.55))
     (stroke (width 0) (type default))
@@
     (stroke (width 0) (type default))
   )
+  (wire (pts (xy 297.18 160.02) (xy 304.8 160.02))
+    (stroke (width 0) (type default))
+  )
   (wire (pts (xy 373.38 54.61) (xy 381 54.61))
     (stroke (width 0) (type default))
   )
+  (wire (pts (xy 304.8 172.72) (xy 304.8 176.53))
+    (stroke (width 0) (type default))
+  )
   (wire (pts (xy 102.87 59.69) (xy 102.87 72.39))
     (stroke (width 0) (type default))
@@
     (stroke (width 0) (type default))
   )
-  (wire (pts (xy 300.99 134.62) (xy 314.96 134.62))
+  (wire (pts (xy 306.07 127) (xy 311.15 127))
     (stroke (width 0) (type default))
   )
@@
     (stroke (width 0) (type default))
   )
+  (wire (pts (xy 320.04 138.43) (xy 326.39 138.43))
+    (stroke (width 0) (type default))
+  )
   (wire (pts (xy 176.53 59.69) (xy 176.53 72.39))
     (stroke (width 0) (type default))
@@
     (stroke (width 0) (type default))
   )
+  (wire (pts (xy 306.07 127) (xy 306.07 134.62))
+    (stroke (width 0) (type default))
+  )
   (wire (pts (xy 52.07 113.03) (xy 52.07 74.93))
     (stroke (width 0) (type default))
@@
     (stroke (width 0) (type default))
   )
+  (wire (pts (xy 297.18 172.72) (xy 297.18 176.53))
+    (stroke (width 0) (type default))
+  )
   (wire (pts (xy 82.55 59.69) (xy 82.55 76.2))
     (stroke (width 0) (type default))
@@
     (stroke (width 0) (type default))
   )
+  (wire (pts (xy 306.07 134.62) (xy 300.99 134.62))
+    (stroke (width 0) (type default))
+  )
   (wire (pts (xy 346.71 187.96) (xy 358.14 187.96))
     (stroke (width 0) (type default))
@@
   )
   (wire (pts (xy 26.67 59.69) (xy 26.67 72.39))
+    (stroke (width 0) (type default))
+  )
+  (wire (pts (xy 300.99 138.43) (xy 309.88 138.43))
     (stroke (width 0) (type default))
   )
@@
     (effects (font (size 1.27 1.27)) (justify left bottom))
   )
+  (label "V+" (at 302.26 160.02 180) (fields_autoplaced)
+    (effects (font (size 1.27 1.27)) (justify right bottom))
+  )
   (label "Row1" (at 224.79 72.39 90) (fields_autoplaced)
     (effects (font (size 1.27 1.27)) (justify left bottom))
@@
   )
   (label "V+" (at 389.89 62.23 180) (fields_autoplaced)
+    (effects (font (size 1.27 1.27)) (justify right bottom))
+  )
+  (label "V+" (at 326.39 138.43 180) (fields_autoplaced)
     (effects (font (size 1.27 1.27)) (justify right bottom))
   )
@@
     )
   )
-  (global_label "SCL" (shape input) (at 314.96 134.62 0)
+  (global_label "SDA" (shape input) (at 297.18 176.53 270) (fields_autoplaced)
+    (effects (font (size 1.27 1.27)) (justify right))
+    (property "Intersheetrefs" "${INTERSHEET_REFS}" (at 297.18 183.0833 90)
+      (effects (font (size 1.27 1.27)) (justify right) hide)
+    )
+  )
+  (global_label "SCL" (shape input) (at 311.15 127 0)
     (effects (font (size 1.27 1.27)) (justify left))
-    (property "Intersheetrefs" "${INTERSHEET_REFS}" (at 314.96 134.62 0)
+    (property "Intersheetrefs" "${INTERSHEET_REFS}" (at 311.15 127 0)
       (effects (font (size 1.27 1.27)) hide)
     )
@@
     (property "Intersheetrefs" "${INTERSHEET_REFS}" (at 340.36 67.31 0)
       (effects (font (size 1.27 1.27)) hide)
+    )
+  )
+  (global_label "SCL" (shape input) (at 304.8 176.53 270) (fields_autoplaced)
+    (effects (font (size 1.27 1.27)) (justify right))
+    (property "Intersheetrefs" "${INTERSHEET_REFS}" (at 304.8 183.0228 90)
+      (effects (font (size 1.27 1.27)) (justify right) hide)
     )
   )
@@
     )
   )
+  (symbol (lib_id "Seismos-sym:Jumper_2_Open") (at 314.96 138.43 0) (unit 1)
+    (in_bom yes) (on_board yes) (dnp no) (fields_autoplaced)
+    (property "Reference" "JP1" (at 314.96 132.08 0)
+      (effects (font (size 1.27 1.27)))
+    )
+    (property "Value" "Jumper_2_Open" (at 314.96 134.62 0)
+      (effects (font (size 1.27 1.27)))
+    )
+    (property "Footprint" "Jumper:SolderJumper-2_P1.3mm_Open_TrianglePad1.0x1.5mm" (at 314.96 138.43 0)
+      (effects (font (size 1.27 1.27)) hide)
+    )
+    (property "Datasheet" "~" (at 314.96 138.43 0)
+      (effects (font (size 1.27 1.27)) hide)
+    )
+    (pin "1")
+    (pin "2")
+    (instances
+      (project "Seismos_5CoreR"
+        (path "/c801d42e-dd94-493e-bd2f-6c3ddad43f55"
+          (reference "JP1") (unit 1)
+        )
+      )
+    )
+  )
   (symbol (lib_id "Seismos-sym:SM10B-SRSS-TB_(LF)(SN)") (at 115.57 53.34 90) (unit 1)
     (in_bom yes) (on_board yes) (dnp no)
@@
     )
   )
+  (symbol (lib_id "Seismos-sym:Resistor") (at 304.8 168.91 0) (unit 1)
+    (in_bom yes) (on_board yes) (dnp no) (fields_autoplaced)
+    (property "Reference" "R2" (at 307.34 167.64 0)
+      (effects (font (size 1.27 1.27)) (justify left))
+    )
+    (property "Value" "R" (at 307.34 170.18 0)
+      (effects (font (size 1.27 1.27)) (justify left))
+    )
+    (property "Footprint" "Resistor_SMD:R_0603_1608Metric_Pad0.98x0.95mm_HandSolder" (at 303.022 168.91 90)
+      (effects (font (size 1.27 1.27)) hide)
+    )
+    (property "Datasheet" "~" (at 304.8 168.91 0)
+      (effects (font (size 1.27 1.27)) hide)
+    )
+    (pin "1")
+    (pin "2")
+    (instances
+      (project "Seismos_5CoreR"
+        (path "/c801d42e-dd94-493e-bd2f-6c3ddad43f55"
+          (reference "R2") (unit 1)
+        )
+      )
+    )
+  )
   (symbol (lib_id "power:GND") (at 337.82 106.68 0) (unit 1)
     (in_bom yes) (on_board yes) (dnp no)
@@
         )
       )
+    )
+  )
+  (symbol (lib_id "Seismos-sym:Resistor") (at 297.18 168.91 0) (unit 1)
+    (in_bom yes) (on_board yes) (dnp no) (fields_autoplaced)
+    (property "Reference" "R1" (at 299.72 167.64 0)
+      (effects (font (size 1.27 1.27)) (justify left))
+    )
+    (property "Value" "R" (at 299.72 170.18 0)
+      (effects (font (size 1.27 1.27)) (justify left))
+    )
+    (property "Footprint" "Resistor_SMD:R_0603_1608Metric_Pad0.98x0.95mm_HandSolder" (at 295.402 168.91 90)
+      (effects (font (size 1.27 1.27)) hide)
+    )
+    (property "Datasheet" "~" (at 297.18 168.91 0)
+      (effects (font (size 1.27 1.27)) hide)
+    )
+    (pin "1")
+    (pin "2")
+    (instances
+      (project "Seismos_5CoreR"
+        (path "/c801d42e-dd94-493e-bd2f-6c3ddad43f55"
+          (reference "R1") (unit 1)
+        )
+      )

Commit message: Fix right encoder button, fix connector refs
Right side encoder was still connected to the 6th column for some
reason... Figures when you copy paste the same board design into a
different project.

Also fixed references for the SH connectors, so it doesn't look weird
Parts:
- J1, J2, J3, J4, J5, J6: value SM09B-SRSS-TB(LF)(SN) -> SM010B-SRSS-TB(LF)(SN)
Connections:
- net Col_In6: no longer SW1.S2
- net Col_InT: now also SW1.S2
Other:
- note added: "Bottom Connectors"
- note removed: "Top Connectors"
Changed lines of the file:
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@@
     (effects (font (size 1.27 1.27)) (justify left top))
   )
-  (text "Top Connectors" (at 73.66 31.75 0)
+  (text "Bottom Connectors" (at 63.5 33.02 0)
     (effects (font (size 10 10)) (justify left bottom))
   )
@@
     (effects (font (size 1.27 1.27)) (justify left bottom))
   )
-  (label "Col_In6" (at 384.81 106.68 180) (fields_autoplaced)
+  (label "Col_InT" (at 384.81 106.68 180) (fields_autoplaced)
     (effects (font (size 1.27 1.27)) (justify right bottom))
   )
@@
       (effects (font (size 1.27 1.27)) (justify left))
     )
-    (property "Value" "SM09B-SRSS-TB(LF)(SN)" (at 242.57 43.18 90)
+    (property "Value" "SM010B-SRSS-TB(LF)(SN)" (at 242.57 43.18 90)
       (effects (font (size 1.27 1.27)) (justify left))
     )
@@
       (effects (font (size 1.27 1.27)) (justify left))
     )
-    (property "Value" "SM09B-SRSS-TB(LF)(SN)" (at 204.47 43.18 90)
+    (property "Value" "SM010B-SRSS-TB(LF)(SN)" (at 204.47 43.18 90)
       (effects (font (size 1.27 1.27)) (justify left))
     )
@@
       (effects (font (size 1.27 1.27)) (justify left))
     )
-    (property "Value" "SM09B-SRSS-TB(LF)(SN)" (at 128.27 43.18 90)
+    (property "Value" "SM010B-SRSS-TB(LF)(SN)" (at 128.27 43.18 90)
       (effects (font (size 1.27 1.27)) (justify left))
     )
@@
       (effects (font (size 1.27 1.27)) (justify left))
     )
-    (property "Value" "SM09B-SRSS-TB(LF)(SN)" (at 52.07 43.18 90)
+    (property "Value" "SM010B-SRSS-TB(LF)(SN)" (at 52.07 43.18 90)
       (effects (font (size 1.27 1.27)) (justify left))
     )
@@
       (effects (font (size 1.27 1.27)) (justify left))
     )
-    (property "Value" "SM09B-SRSS-TB(LF)(SN)" (at 166.37 43.18 90)
+    (property "Value" "SM010B-SRSS-TB(LF)(SN)" (at 166.37 43.18 90)
       (effects (font (size 1.27 1.27)) (justify left))
     )
@@
       (effects (font (size 1.27 1.27)) (justify left))
     )
-    (property "Value" "SM09B-SRSS-TB(LF)(SN)" (at 90.17 43.18 90)
-      (effects (font (size 1.27 1.27)) (justify left))
-    )
+    (property "Value" "SM010B-SRSS-TB(LF)(SN)" (at 90.17 43.18 90)
+      (effects (font (size 1.27 1.27)) (justify left))
+    )

Commit message: Added 74HC595A support, new release
New PCB versions supporting shift register.
Another JST SH connector is added to expose 2 spare pins.

Footprints for microcontroller were updated using modified footprint from library.
Original variants updated to these new footprints with some fixes as well.
Parts:
- J7: value SM09B-SRSS-TB(LF)(SN) -> SM10B-SRSS-TB_(LF)(SN)
- U1: footprint keyboard_reversible:ProMicro -> Seismos-libs:keebRev-onesided_ProMicro
Connections:
- net GND: now also SW1.MP
Changed lines of the file:
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@@
+    (stroke (width 0) (type default))
+  )
+  (wire (pts (xy 373.38 96.52) (xy 368.3 96.52))
     (stroke (width 0) (type default))
   )
@@
     (pin "B")
     (pin "C")
+    (pin "MP")
     (pin "S1")
     (pin "S2")
@@
     )
   )
-  (symbol (lib_name "GND_1") (lib_id "power:GND") (at 74.93 130.81 0) (mirror y) (unit 1)
+  (symbol (lib_id "power:GND") (at 74.93 130.81 0) (mirror y) (unit 1)
     (in_bom yes) (on_board yes) (dnp no)
     (property "Reference" "#PWR023" (at 74.93 137.16 0)
@@
     )
   )
-  (symbol (lib_name "GND_1") (lib_id "power:GND") (at 227.33 62.23 0) (mirror y) (unit 1)
+  (symbol (lib_id "power:GND") (at 227.33 62.23 0) (mirror y) (unit 1)
     (in_bom yes) (on_board yes) (dnp no)
     (property "Reference" "#PWR026" (at 227.33 68.58 0)
@@
     )
   )
-  (symbol (lib_name "GND_1") (lib_id "power:GND") (at 74.93 62.23 0) (mirror y) (unit 1)
+  (symbol (lib_id "power:GND") (at 74.93 62.23 0) (mirror y) (unit 1)
     (in_bom yes) (on_board yes) (dnp no)
     (property "Reference" "#PWR03" (at 74.93 68.58 0)
@@
       (effects (font (size 1.27 1.27)))
     )
-    (property "Footprint" "keyboard_reversible:ProMicro" (at 355.6 66.04 0)
+    (property "Footprint" "Seismos-libs:keebRev-onesided_ProMicro" (at 355.6 66.04 0)
       (effects (font (size 1.27 1.27)) hide)
     )
@@
     )
   )
-  (symbol (lib_name "GND_1") (lib_id "power:GND") (at 342.9 172.72 270) (mirror x) (unit 1)
+  (symbol (lib_id "power:GND") (at 342.9 172.72 270) (mirror x) (unit 1)
     (in_bom yes) (on_board yes) (dnp no)
     (property "Reference" "#PWR020" (at 336.55 172.72 0)
@@
     )
   )
-  (symbol (lib_name "GND_1") (lib_id "power:GND") (at 36.83 62.23 0) (mirror y) (unit 1)
+  (symbol (lib_id "power:GND") (at 373.38 96.52 90) (mirror x) (unit 1)
+    (in_bom yes) (on_board yes) (dnp no)
+    (property "Reference" "#PWR03" (at 379.73 96.52 0)
+      (effects (font (size 1.27 1.27)) hide)
+    )
+    (property "Value" "GND" (at 376.6312 96.647 90)
+      (effects (font (size 1.27 1.27)) (justify right))
+    )
+    (property "Footprint" "" (at 373.38 96.52 0)
+      (effects (font (size 1.27 1.27)) hide)
+    )
+    (property "Datasheet" "" (at 373.38 96.52 0)
+      (effects (font (size 1.27 1.27)) hide)
+    )
+    (pin "1")
+    (instances
+      (project "KeysOnRails_Carrier1"
+        (path "/a6dae978-c8fe-4bbf-835b-e2bd64164dfb"
+          (reference "#PWR03") (unit 1)
+        )
+      )
+      (project "Seismos_5CoreR"
+        (path "/c801d42e-dd94-493e-bd2f-6c3ddad43f55"
+          (reference "#PWR029") (unit 1)
+        )
+      )
+    )
+  )
+  (symbol (lib_id "power:GND") (at 36.83 62.23 0) (mirror y) (unit 1)
     (in_bom yes) (on_board yes) (dnp no)
     (property "Reference" "#PWR01" (at 36.83 68.58 0)
@@
       (effects (font (size 1.27 1.27)) (justify left))
     )
-    (property "Value" "SM09B-SRSS-TB(LF)(SN)" (at 372.11 187.96 90)
+    (property "Value" "SM10B-SRSS-TB_(LF)(SN)" (at 372.11 187.96 90)
       (effects (font (size 1.27 1.27)) (justify left))
     )
@@
     )
   )
-  (symbol (lib_name "GND_1") (lib_id "power:GND") (at 113.03 62.23 0) (mirror y) (unit 1)
+  (symbol (lib_id "power:GND") (at 113.03 62.23 0) (mirror y) (unit 1)
     (in_bom yes) (on_board yes) (dnp no)
     (property "Reference" "#PWR06" (at 113.03 68.58 0)
@@
     )
   )
-  (symbol (lib_name "GND_1") (lib_id "power:GND") (at 189.23 62.23 0) (mirror y) (unit 1)
+  (symbol (lib_id "power:GND") (at 189.23 62.23 0) (mirror y) (unit 1)
     (in_bom yes) (on_board yes) (dnp no)
     (property "Reference" "#PWR025" (at 189.23 68.58 0)
@@
     )
   )
-  (symbol (lib_name "GND_1") (lib_id "power:GND") (at 151.13 62.23 0) (mirror y) (unit 1)
+  (symbol (lib_id "power:GND") (at 151.13 62.23 0) (mirror y) (unit 1)
     (in_bom yes) (on_board yes) (dnp no)
     (property "Reference" "#PWR016" (at 151.13 68.58 0)

Commit message: HOTFIX, power switch bridges to ground
Connections:
- net GND: no longer U2.L1
