File: pcbs/Core PCBs (Mantles)/5 Key Core (Using Shift Register)/Seismos_5CoreLShift/Seismos_5CoreLShift.kicad_sch (KiCad schematic)
At the start: 26 parts, among them IC1 74HC595, J1 SM010B-SRSS-TB(LF)(SN), J10 SM10B-SRSS-TB_(LF)(SN), J2 SM010B-SRSS-TB(LF)(SN), J3 SM010B-SRSS-TB(LF)(SN), J4 SM010B-SRSS-TB(LF)(SN), J5 SM010B-SRSS-TB(LF)(SN), J6 SM010B-SRSS-TB(LF)(SN), J7 SM10B-SRSS-TB_(LF)(SN), J8 MJ-4PP-9-Lily58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

Commit message: HOTFIX, power switch bridges to ground
Connections:
- net GND: no longer U2.L2
